File: hardware/kicad/485toSDI12/485toSDI12.kicad_sch (KiCad schematic)
At the start: 38 parts, among them J1 Conn_01x04, Q1 2N7002, Q2 MMBT3906, U1 STM32G431C8Tx, U2 AP2112K-3.3, U3 74LVC1G125SE-7, U4 SP3485EN, Y1 8MHz

Commit message: Initial Dajilog Zephyr device platform
Parts:
- removed C10, C11, C9: 4.7uF, Resistor_SMD:R_0805_2012Metric_Pad1.20x1.40mm_HandSolder, symbol Device:C_Small
- removed C12: 100nF, symbol Device:C_Small
- removed C4, C6, C7, C8: 100nF, Resistor_SMD:R_0805_2012Metric_Pad1.20x1.40mm_HandSolder, symbol Device:C_Small
- removed D1: BZT52Bxx, Diode_SMD:D_SOD-123F, symbol Diode:BZT52Bxx
- removed FB1: FerriteBead, symbol Device:FerriteBead
- removed L1: 10uH, symbol Device:L
- removed Q1: 2N7002, Package_TO_SOT_SMD:SOT-23, symbol Transistor_FET:2N7002
- removed Q2: MMBT3906, Package_TO_SOT_SMD:SOT-23, symbol Transistor_BJT:MMBT3906
- removed R1: 10k, Resistor_SMD:R_0805_2012Metric_Pad1.20x1.40mm_HandSolder, symbol Device:R
- removed R10, R7: 100/J, Resistor_SMD:R_0805_2012Metric_Pad1.20x1.40mm_HandSolder, symbol Device:R_US
- removed R11, R9: 2.2K/J, Resistor_SMD:R_0805_2012Metric_Pad1.20x1.40mm_HandSolder, symbol Device:R_US
- removed R12, R8: 0/J, Resistor_SMD:R_0805_2012Metric_Pad1.20x1.40mm_HandSolder, symbol Device:R_US
- removed R14, R15, R17: 10K/J, Resistor_SMD:R_0805_2012Metric_Pad1.20x1.40mm_HandSolder, symbol Device:R_US
- removed R2: 1k, Resistor_SMD:R_0805_2012Metric_Pad1.20x1.40mm_HandSolder, symbol Device:R
- removed R3: 4.7k, Resistor_SMD:R_0805_2012Metric_Pad1.20x1.40mm_HandSolder, symbol Device:R
- removed R4, R6: 510, Resistor_SMD:R_0805_2012Metric_Pad1.20x1.40mm_HandSolder, symbol Device:R
- removed R5: 200k, symbol Device:R
- removed U2: AP2112K-3.3, Package_TO_SOT_SMD:SOT-23-5, symbol Regulator_Linear:AP2112K-3.3
- removed U3: 74LVC1G125SE-7, 74LVC1G125SE-7:SOT65P210X110-5N, symbol 74LVC1G1:74LVC1G125SE-7
- removed U4: SP3485EN, Package_SO:SOIC-8_3.9x4.9mm_P1.27mm, symbol Interface_UART:SP3485EN
- removed Y1: 8MHz, symbol Device:Crystal
- added C16, C21, C31: 100nF, Resistor_SMD:R_0805_2012Metric_Pad1.20x1.40mm_HandSolder, symbol Device:C_Small
- added C33, C48, C50: 1uF, Resistor_SMD:R_0805_2012Metric_Pad1.20x1.40mm_HandSolder, symbol Device:C_Small
- added D19: 1N5819, Diode_SMD:D_SOD-323, symbol Diode:1N5819WS
- added D3: PESD3V3S1UB, Diode_SMD:D_SOD-923, symbol Diode:ESD9B3.3ST5G
- added F1: MF-PSMF050X-2, Capacitor_SMD:C_0805_2012Metric_Pad1.18x1.45mm_HandSolder, symbol Device:Polyfuse
- added FB5: 600Ω @ 100MHz, Inductor_SMD:L_0805_2012Metric_Pad1.05x1.20mm_HandSolder, symbol Device:FerriteBead_Small
- added R27, R28: 10K/J, Resistor_SMD:R_0805_2012Metric, symbol Device:R_US
- added SW2: NRST, Button_Switch_SMD:SW_Tactile_SPST_NO_Straight_CK_PTS636Sx25SMTRLFS, symbol Switch:SW_Push
- added U9: USBLC6-2SC6, Package_TO_SOT_SMD:SOT-23-6, symbol Power_Protection:USBLC6-2SC6
- added USB1: USB_C_Receptacle_USB2.0_16P, Connector_USB:USB_C_Receptacle_G-Switch_GT-USB-7010ASV, symbol Connector:USB_C_Receptacle_USB2.0_16P
- added Y2: 8Mhz, Crystal:Crystal_SMD_HC49-SD, symbol Device:Crystal
- J1: value Conn_01x04 -> Debug; footprint (none) -> Connector_PinHeader_2.54mm:PinHeader_1x04_P2.54mm_Vertical
Connections:
- net +3.3V: now also C16.2, C21.2, C33.2, C48.2, FB5.1
- net +3.3VA: now also C50.2, FB5.2
- net +5V: now also D19.1 (K), U9.5 (VBUS)
- net GND: now also C16.1, C21.1, C31.1, C33.1, C48.1, C50.1, D3.2 (A2), R27.2, R28.2, SW2.1, U9.2 (GND), USB1.A1 (GND), USB1.A12 (GND), USB1.B1 (GND), USB1.B12 (GND), USB1.SH (SHIELD); no longer U1.29 (PB15)
- net OE: now also U1.26 (PB12)
- net OSC_IN: now also Y2.2
- net OSC_OUT: now also Y2.1
- net SPI_SCLK: now reaches U1.13 (PA5)
- net SPI_DOUT: now reaches U1.14 (PA6)
- net SPI_PWDN: now reaches U1.15 (PA7)
- net TXD3: now reaches U1.22 (PB10)
- net RXD3: now reaches U1.25 (PB11)
- net I2C3_SCL: now reaches U1.30 (PA8)
- net USB D-: now reaches U1.33 (PA11)
- net USB D-: now also U9.6 (I/O1)
- net USB D+: now reaches U1.34 (PA12)
- net USB D+: now also U9.4 (I/O2)
- net I2C1_SCL: now reaches U1.39 (PA15)
- net DO2: now reaches U1.40 (PB3)
- net DO1: now reaches U1.41 (PB4)
- net I2C3_SDA: now reaches U1.42 (PB5)
- net I2C1_SDA: now reaches U1.44 (PB7)
- net CANFD_RX: now reaches U1.45 (PB8)
- net CANFD_TX: now reaches U1.46 (PB9)
- net at C3.2, U1.7 (PG10-NRST): now also D3.1 (A1), SW2.2
- new net: R27.1, USB1.A5 (CC1)
- new net: U9.3 (I/O2), USB1.A6 (D+), USB1.B6 (D+)
- new net: U9.1 (I/O1), USB1.A7 (D-), USB1.B7 (D-)
- new net: R28.1, USB1.B5 (CC2)
- new net: C31.2, D19.2 (A), F1.2
- new net 485_EN: U1.29 (PB15)
- new net VUSB: F1.1, USB1.A4 (VBUS), USB1.A9 (VBUS), USB1.B4 (VBUS), USB1.B9 (VBUS)
Other:
- added sheet ADC, CURRENT_LOOP (ADC_4_20MA.kicad_sch)
- added sheet Relay_out Sheet (Relay_out.kicad_sch)
- added sheet interface (interface.kicad_sch)
- added sheet interface-sdi12-sbus (interface-sdi12-sbus.kicad_sch)
- added sheet power (power.kicad_sch)
- note added: "crystal"
- note removed: "3.3V Reguator"
- note removed: "OSCILATTOR"
- note removed: "RS485"
- note removed: "SDI12 slave"
- moved on the sheet: C1, C2, J1
