File: hardware/kicad/agmo/Tractor_Ignition_Control/TIC/MCU.kicad_sch (KiCad schematic)
At the start: 42 parts, among them CN1 CAN, J1 Debug, J4 Conn_01x06, SW2 NRST, U1 STM32G431C8Tx, U15 π142M31, U8 TJA1051T-3, U9 USBLC6-2SC6, Y2 8Mhz

Commit message: feat(hardware): update TIC KiCad design and fabrication files
Parts:
- added R58: 10k, Resistor_SMD:R_0805_2012Metric, symbol Device:R_US
- FL1: now not fitted; now left out of the parts list
Connections:
- net DI_3 is gone; now on net DO5: U1.31 (PA9)
- net CAN_H: now also U8.7 (CANH); no longer FL1.4
- net CAN_L: now also U8.6 (CANL); no longer FL1.3
- net GND: now also R58.1
- net at FL1.1: no longer U8.7 (CANH)
- net at FL1.2: no longer U8.6 (CANL)
- net ISO_DO5: now reaches U15.14 (B1)
- net DO5: now reaches U15.3 (A1)
- net DO5: now also R58.2
