File: hardware/kicad/agmo/Tractor_Ignition_Control/TIC/TIC.kicad_pcb (KiCad board)
At the start: 2 copper layers, 92 x 87 mm, 146 parts, among them CN1 CAN, CN6 power, J1 Debug, J2 Screw_Terminal_01x06, J3 Screw_Terminal_01x04, K1 G5V-2-H1, K2 G5V-2-H1, K3 G5V-2-H1, K4 G5V-2-H1, Q1 IRLML6344, Q2 SQ2361CEES-T1_GE3, Q5 IRLML6344, Q6 IRLML6344, Q7 IRLML6344, SW2 NRST, U1 STM32G431C8Tx, U12 AP2112K-3.3, U14 B0505S-3W, U15 π142M31, U17 π140U31, U18 π140U31, U2 AP2112K-3.3, U3 TLP293, U4 TLP293, U5 TPS5430DDA, U6 TLP293, U8 TJA1051T-3, U9 USBLC6-2SC6, Y2 8Mhz

Commit message: feat(hardware): update TIC KiCad design and fabrication files
Parts:
- removed C10: 22nF, Capacitor_SMD:C_0805_2012Metric_Pad1.18x1.45mm_HandSolder
- removed R10, R9: 4.7k, Resistor_SMD:R_0805_2012Metric
- removed R11: 100, Resistor_SMD:R_0805_2012Metric
- removed R12: 10k, Resistor_SMD:R_0805_2012Metric
- added C19: 220nF/100V, Capacitor_SMD:C_1812_4532Metric, F.Cu at (94.2, 145.0)
- added C23: 4.7uF/100V, Capacitor_SMD:C_1812_4532Metric, F.Cu at (94.2, 149.9)
- added C24: 100nF/10V, Capacitor_SMD:C_0805_2012Metric_Pad1.18x1.45mm_HandSolder, F.Cu at (101.2, 158.8)
- added C25: 4.7uF/100V, Capacitor_SMD:C_1812_4532Metric, F.Cu at (94.2, 154.9)
- added C26: 220uF/50V, Capacitor_SMD:CP_Elec_10x10, F.Cu at (83.8, 162.9)
- added C45: 1uF/V10, Capacitor_SMD:C_0805_2012Metric, F.Cu at (101.0, 167.9)
- added C58: 22uF/25V, Capacitor_SMD:C_0805_2012Metric_Pad1.18x1.45mm_HandSolder, F.Cu at (101.2, 161.8)
- added C59: 22uF/25V, Capacitor_SMD:C_0805_2012Metric_Pad1.18x1.45mm_HandSolder, F.Cu at (101.2, 164.9)
- added CN7: power, Connector_Phoenix_MSTB:PhoenixContact_MSTBA_2,5_2-G-5,08_1x02_P5.08mm_Horizontal, F.Cu at (81.0, 145.9)
- added D17: SMCJ33CA, Diode_SMD:D_SMA, F.Cu at (94.7, 164.2)
- added D20: LED RED, LED_SMD:LED_0805_2012Metric, F.Cu at (112.2, 144.0)
- added D21: LED RED, LED_SMD:LED_0805_2012Metric, F.Cu at (112.2, 147.0)
- added D22: LED RED, LED_SMD:LED_0805_2012Metric, F.Cu at (112.2, 150.1)
- added D23: LED RED, LED_SMD:LED_0805_2012Metric, F.Cu at (112.2, 153.1)
- added D30: LED RED, LED_SMD:LED_0805_2012Metric, F.Cu at (102.0, 64.4)
- added F3: 0466005.NRHF, Fuse:Fuse_1206_3216Metric_Pad1.42x1.75mm_HandSolder, F.Cu at (93.7, 168.1)
- added L3: 10uH, Inductor_SMD:L_APV_APH0630, F.Cu at (102.7, 146.6)
- added Q4: SQ2361CEES-T1_GE3, Package_TO_SOT_SMD:SOT-23, F.Cu at (106.9, 62.6)
- added R33: 47k, Resistor_SMD:R_0805_2012Metric, F.Cu at (108.1, 68.0)
- added R35: 24.9k, Resistor_SMD:R_0805_2012Metric, F.Cu at (105.8, 158.8)
- added R36: 100k, Resistor_SMD:R_0805_2012Metric, F.Cu at (105.8, 161.8)
- added R38: 10k, Resistor_SMD:R_0805_2012Metric, F.Cu at (105.8, 164.7)
- added R56: 1k, Resistor_SMD:R_0805_2012Metric, F.Cu at (99.7, 71.1)
- added R57: 4.7k, Resistor_SMD:R_0805_2012Metric, F.Cu at (102.0, 62.2)
- added R58: 10k, Resistor_SMD:R_0805_2012Metric, F.Cu at (75.5, 65.8)
- added U7: LMR36510ADDA, Package_SO:Texas_HTSOP-8-1EP_3.9x4.9mm_P1.27mm_EP2.95x4.9mm_Mask2.4x3.1mm_ThermalVias, F.Cu at (102.5, 154.0)
- D10: value SMAJ33A -> SS310
- D11: value 1N4148W -> BZT52C16
- moved D10 95.5 mm to (94.7, 159.6)
- moved U6 1.07 mm to (105.3, 71.3), turned to 0 degrees
- moved D11 0.92 mm to (107.4, 65.7), turned to 180 degrees
- moved USB1 0.60 mm to (51.2, 89.4)
- moved D19 0.55 mm to (62.9, 92.4)
- moved C31 0.55 mm to (59.6, 93.1)
- moved F1 0.55 mm to (59.6, 91.0)
- moved R27 0.55 mm to (59.5, 82.7)
- moved R28 0.55 mm to (59.5, 88.8)
- moved U9 0.55 mm to (59.8, 85.7)
- moved U14 0.40 mm to (75.0, 125.1)
- moved CN6 0.40 mm to (61.7, 121.5)
- moved Q2 0.40 mm to (50.6, 113.8)
- moved K1 0.40 mm to (92.0, 98.0)
- moved K2 0.40 mm to (104.0, 98.0)
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- renumbered RESTART to START
Connections:
- C7 pad 2: /input Sheet/D_COM -> D_COM
- C8 pad 2: /input Sheet/D_COM -> D_COM
- D1 pad 2: /input Sheet/D_COM -> D_COM
- D10 pad 1: /input Sheet/D_IN3 -> Net-(D10-K)
- D10 pad 2: /input Sheet/D_COM -> Net-(D10-A)
- D11 pad 1: Net-(D11-K) -> D_IN1
- D11 pad 2: /input Sheet/D_COM -> Net-(D11-A)
- D4 pad 1: /input Sheet/D_IN1 -> D_IN1
- D4 pad 2: /input Sheet/D_COM -> D_COM
- D5 pad 2: /input Sheet/D_COM -> D_COM
- D8 pad 2: /input Sheet/D_COM -> D_COM
- J3 pad 1: /input Sheet/D_IN1 -> D_IN1
- J3 pad 3: /input Sheet/D_IN3 -> D_COM
- J3 pad 4: /input Sheet/D_COM -> D_OUT5
- R1 pad 1: /input Sheet/D_IN1 -> D_IN1
- R40 pad 1: /MCU/CAN_H -> /MCU/CAN_L
- R40 pad 2: /MCU/CAN_L -> /MCU/CAN_H
- U1 pad 31: DI_3 -> DO5
- U15 pad 14: unconnected-(U15-B1-Pad14) -> ISO_DO5
- U15 pad 3: unconnected-(U15-A1-Pad3) -> DO5
- U17 pad 12: DI_3 -> unconnected-(U17-B3-Pad12)
- U17 pad 5: /input Sheet/ISO_DI3 -> unconnected-(U17-A3-Pad5)
- U3 pad 2: /input Sheet/D_COM -> D_COM
- U4 pad 2: /input Sheet/D_COM -> D_COM
- U6 pad 1: Net-(D11-K) -> Net-(R56-Pad2)
- U6 pad 2: /input Sheet/D_COM -> SGND
- U6 pad 3: SGND -> D_COM
- U6 pad 4: Net-(R11-Pad2) -> Net-(D11-A)
Routing:
- net ISO_DO5: track 0.00 -> 32.6 mm
- net ISO_3.3V: track 144.5 -> 123.1 mm, vias 6 -> 7
- net DO5: track 0.00 -> 20.9 mm
- net /input Sheet/D_IN3: track 20.2 -> 0.00 mm
- net D_IN1: track 0.00 -> 19.0 mm, vias 0 -> 5
- net /input Sheet/ISO_DI3: track 18.0 -> 0.00 mm
- net DI_3: track 12.5 -> 0.00 mm
- net /input Sheet/D_IN1: track 11.6 -> 0.00 mm
- net Net-(D11-A): track 0.00 -> 11.1 mm
- net Net-(D11-K): track 10.8 -> 0.00 mm
- net Net-(R11-Pad2): track 2.64 -> 0.00 mm
- net Net-(R56-Pad2): track 0.00 -> 2.59 mm
- net Net-(D30-A): track 0.00 -> 2.23 mm
- net Net-(R10-Pad1): track 1.70 -> 0.00 mm
- net BAT+: track 148.3 -> 147.3 mm
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- added copper zone on B.Cu, net D_COM
- added copper zone on F.Cu, net D_COM
- added copper zone on B.Cu, net D_IN1
- added copper zone on F.Cu, net D_IN1
- added copper zone on F.Cu, net D_OUT5
- removed copper zone on B.Cu, net /input Sheet/D_COM
- removed copper zone on F.Cu, net /input Sheet/D_COM
Other:
- board text added: "AGMO_TIC 09.22_VER.02"
- board text added: "DI_3 DI_G DI_2 DI_1"
- board text removed: "AGMO_TIC 2026.08.07_VER.01"
- board text removed: "DI_G DI_3 DI_2 DI_1"
