File: hardware/kicad/agmo/Tractor_Ignition_Control/TIC/power.kicad_sch (KiCad schematic)
At the start: 38 parts, among them CN6 power, Q2 SQ2361CEES-T1_GE3, U12 AP2112K-3.3, U14 B0505S-3W, U2 AP2112K-3.3, U5 TPS5430DDA

Commit message: feat(hardware): update TIC KiCad design and fabrication files
Parts:
- added C19: 220nF/100V, Capacitor_SMD:C_0603_1608Metric, symbol Device:C
- added C23, C25: 4.7uF/100V, Capacitor_SMD:C_1210_3225Metric, symbol Device:C
- added C24: 100nF/10V, Capacitor_SMD:C_0805_2012Metric_Pad1.18x1.45mm_HandSolder, symbol Device:C
- added C26: 220uF/50V, Capacitor_SMD:CP_Elec_10x10, symbol Device:C_Polarized_US
- added C45: 1uF/V10, Capacitor_SMD:C_0805_2012Metric, symbol Device:C
- added C58, C59: 22uF/25V, Capacitor_SMD:C_0805_2012Metric_Pad1.18x1.45mm_HandSolder, symbol Device:C
- added CN7: power, Connector_Phoenix_MSTB:PhoenixContact_MSTBA_2,5_2-G-5,08_1x02_P5.08mm_Horizontal, symbol Connector_Generic:Conn_01x02
- added D10: SS310, Diode_SMD:D_SMA, symbol Diode:SS310
- added D17: SMCJ33CA, Diode_SMD:D_SMC, symbol Diode:SMAJ24A
- added F3: 0466005.NRHF, Fuse:Fuse_1206_3216Metric_Pad1.42x1.75mm_HandSolder, symbol Device:Fuse
- added L3: 10uH, Inductor_SMD:L_APV_APH0630, symbol Device:L_Iron
- added R35: 24.9k, Resistor_SMD:R_0805_2012Metric, symbol Device:R_US
- added R36: 100k, Resistor_SMD:R_0805_2012Metric, symbol Device:R_US
- added R38: 10k, Resistor_SMD:R_0805_2012Metric, symbol Device:R_US
- added TP1: TestPoint, symbol Connector:TestPoint
- added U7: LMR36510ADDA, Package_SO:Texas_HTSOP-8-1EP_3.9x4.9mm_P1.27mm_EP2.95x4.9mm_Mask2.4x3.1mm_ThermalVias, symbol Regulator_Switching:LMR36510ADDA
- R47: now not fitted
Connections:
- net +5V: now also C58.1, C59.1, L3.2, R36.1, R38.2
- net BAT+: now also CN7.2 (Pin_2), F3.1
- net GND: now also C19.2, C23.2, C25.2, C26.2, C45.2, C58.2, C59.2, CN7.1 (Pin_1), D17.2 (A2), R35.2, U7.1 (PGND), U7.9 (PAD)
- new net: C19.1, C23.1, C25.1, C26.1, D10.1 (K), U7.2 (VIN), U7.3 (EN)
- new net: D10.2 (A), D17.1 (A1), F3.2
- new net: R38.1, TP1.1, U7.4 (PG)
- new net: C45.1, U7.6 (VCC)
- new net: R35.1, R36.2, U7.5 (FB)
- new net: C24.1, L3.1, U7.8 (SW)
- new net: C24.2, U7.7 (BOOT)
Other:
- note added: "5V / 2A"
- moved on the sheet: C11, C32, C38, C39, C4, C40, C41, C42, C6, C9, D16, D18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
